File: Low voltage/Relay.sch (EAGLE design)
At the start: 9 parts, among them T1 2N1613

Commit message: board layout
Parts:
- removed R1: 1k, resistor:R-US_R2012
Connections:
- removed net N$3: LED1.A, R1.2
- net N$2: now also LED1.A; no longer R1.1
Changed lines of the file:
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@@
 <parts>
 <part name="U$1" library="SRD-05VDC-SL-C" deviceset="RELAY" device="PTH"/>
-<part name="R1" library="resistor" deviceset="R-US_" device="R2012" value="1k"/>
 <part name="LED1" library="led" deviceset="LED" device="3MM"/>
 <part name="T1" library="transistor" deviceset="2N1613" device=""/>
@@
 <instances>
 <instance part="U$1" gate="G$1" x="121.92" y="38.1"/>
-<instance part="R1" gate="G$1" x="30.48" y="63.5"/>
 <instance part="LED1" gate="G$1" x="43.18" y="63.5" rot="R90"/>
 <instance part="T1" gate="G$1" x="109.22" y="63.5"/>
@@
 </busses>
 <nets>
-<net name="N$3" class="0">
-<segment>
-<pinref part="R1" gate="G$1" pin="2"/>
-<pinref part="LED1" gate="G$1" pin="A"/>
-<wire x1="35.56" y1="63.5" x2="40.64" y2="63.5" width="0.1524" layer="91"/>
-<junction x="35.56" y="63.5"/>
-<junction x="40.64" y="63.5"/>
-</segment>
-</net>
 <net name="N$2" class="0">
 <segment>
 <pinref part="U$3" gate="G$1" pin="GPIO2"/>
-<wire x1="-2.54" y1="63.5" x2="25.4" y2="63.5" width="0.1524" layer="91"/>
+<wire x1="-2.54" y1="63.5" x2="35.56" y2="63.5" width="0.1524" layer="91"/>
 <junction x="-2.54" y="63.5"/>
-<pinref part="R1" gate="G$1" pin="1"/>
-<junction x="25.4" y="63.5"/>
+<pinref part="LED1" gate="G$1" pin="A"/>
+<wire x1="35.56" y1="63.5" x2="38.1" y2="63.5" width="0.1524" layer="91"/>
+<junction x="40.64" y="63.5"/>
+<wire x1="38.1" y1="63.5" x2="40.64" y2="63.5" width="0.1524" layer="91"/>
 </segment>
 </net>
